Commit message: Fixed urdf

File: src/p3at_bringup/urdf/pioneer.urdf.xacro (robot description, xacro)
@@ -135,5 +135,5 @@
     </collision>
   </link>
-  <joint name="p3at_front_left_wheel_joint" type="continuous">
+  <joint name="p3at_front_left_wheel_joint" type="fixed">
     <axis xyz="0 1 0"/>
     <anchor xyz="0 0 0"/>
@@ -222,5 +222,5 @@
     </collision>
   </link>
-  <joint name="p3at_front_right_wheel_joint" type="continuous">
+  <joint name="p3at_front_right_wheel_joint" type="fixed">
     <axis xyz="0 1 0"/>
     <anchor xyz="0 0 0"/>
@@ -309,5 +309,5 @@
     </collision>
   </link>
-  <joint name="p3at_back_left_wheel_joint" type="continuous">
+  <joint name="p3at_back_left_wheel_joint" type="fixed">
     <axis xyz="0 1 0"/>
     <anchor xyz="0 0 0"/>
@@ -396,5 +396,5 @@
     </collision>
   </link>
-  <joint name="p3at_back_right_wheel_joint" type="continuous">
+  <joint name="p3at_back_right_wheel_joint" type="fixed">
     <axis xyz="0 1 0"/>
     <anchor xyz="0 0 0"/>
@@ -454,9 +454,19 @@
   <link name="cam_optical_link"></link>
   <!-- IMU -->
-  <link name="imu_link"/>
+  <link name="imu_link">
+    <visual>
+      <origin xyz="0 0 0" rpy="0 0 0"/>
+      <geometry>
+        <box size="0.05 0.05 0.005"/>
+      </geometry>
+      <material name="imu">
+        <color rgba="0 1.0 1.0 1.0"/>
+      </material>
+    </visual>
+  </link>
   <joint name="imu_top_joint" type="fixed">
     <parent link="top_plate" />
     <child link="imu_link" />
-    <origin xyz="0.1 0.1 0.01" rpy="0 0 0"/>
+    <origin xyz="0.1 0.1 0.005" rpy="0 0 0"/>
   </joint>
 </robot>
